File: schematics_&_pcb/poncho.sch (KiCad schematic (older format))
At the start: 21 parts, among them J1 TB_1X2, J2 TB_1X2, J3 TB_1X2, J4 TB_1X3, J5 TB_1X3, J6 TB_1X3, J7 TB_1X3, P1 CONN_20X2, P2 CONN_20X2, P3 ESP8266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

Commit message: Poncho modificado a dos capas.
Parts:
- P3: footprint Housings_DIP:DIP-8_W7.62mm_LongPads -> Pin_Headers:Pin_Header_Straight_2x04
Changed lines of the file:
@@
 EESchema Schematic File Version 2
 LIBS:poncho-rescue
-LIBS:power
-LIBS:device
-LIBS:transistors
-LIBS:conn
-LIBS:linear
-LIBS:regul
-LIBS:74xx
-LIBS:cmos4000
-LIBS:adc-dac
-LIBS:memory
-LIBS:xilinx
-LIBS:microcontrollers
-LIBS:dsp
-LIBS:microchip
-LIBS:analog_switches
-LIBS:motorola
-LIBS:texas
-LIBS:intel
-LIBS:audio
-LIBS:interface
-LIBS:digital-audio
-LIBS:philips
-LIBS:display
-LIBS:cypress
-LIBS:siliconi
-LIBS:opto
-LIBS:atmel
-LIBS:contrib
-LIBS:valves
 LIBS:stepper drivers
 LIBS:terminal_block
@@
 F 0 "P3" H 8250 1200 60  0000 C CNN
 F 1 "ESP8266" V 8250 950 50  0000 C CNN
-F 2 "Housings_DIP:DIP-8_W7.62mm_LongPads" H 8250 950 60  0001 C CNN
+F 2 "Pin_Headers:Pin_Header_Straight_2x04" H 8250 950 60  0001 C CNN
 F 3 "" H 8250 950 60  0000 C CNN
 	1    8250 950

Commit message: Pines de la capa superior corregidos, cambio GPIO2 a GPIO6 para L293D, diodos agregados para alimentación y recepción, encoders con TCST2103 agregados, boton de encendido y regulador agregados.
Parts:
- removed D1, D2: LED, LEDs:LED-5MM, symbol LED-RESCUE-poncho
- removed Q1, Q2: NPN-PHOTO-2, modules:PHOTOTRANS-5MM, symbol NPN-PHOTO-2
- added 78051: LM7805reg, poncho_educiaa:LM7805, symbol LM7805reg
- added D3, D4: LED, LEDs:LED-3MM, symbol LED
- added J8, J9: TB_1X2, Pin_Headers:Pin_Header_Straight_1x02, symbol TB_1X2
- added R5, R6: R, Resistors_ThroughHole:Resistor_Horizontal_RM10mm, symbol R
- added R7: 1k, Resistors_ThroughHole:Resistor_Horizontal_RM10mm, symbol R
- added R8: 680, Resistors_ThroughHole:Resistor_Horizontal_RM10mm, symbol R
- added SW1: 6pin_switch, poncho_educiaa:6pin_switch, symbol 6pin_switch
- added TCST1, TCST2: TCST2103, library:TCST2103, symbol TCST2103
- R1: value 4700 -> 180
- R2: value 100 -> 1k
- R3: value 4700 -> 680
- R4: value 100 -> 180
Connections:
- wire segments 307 -> 332
- no-connect marks 2 -> 6
Other:
- moved on the sheet: J4

Commit message: Borneras agregadas.
Parts:
- J1, J2, J3, J8, J9: footprint Pin_Headers:Pin_Header_Straight_1x02 -> poncho_educiaa:bornera1x2
- J4, J5, J6, J7: footprint Pin_Headers:Pin_Header_Straight_1x03 -> poncho_educiaa:bornera1x3
- renumbered 78051 to 780511
Changed lines of the file:
@@
 F 0 "J1" H 5950 3450 60  0000 C CNN
 F 1 "TB_1X2" H 6000 2850 60  0000 C CNN
-F 2 "Pin_Headers:Pin_Header_Straight_1x02" H 5900 3200 60  0001 C CNN
+F 2 "poncho_educiaa:bornera1x2" H 5900 3200 60  0001 C CNN
 F 3 "" H 5900 3200 60  0000 C CNN
 	1    5950 3150
@@
 F 0 "J2" H 11000 3450 60  0000 C CNN
 F 1 "TB_1X2" H 11050 2850 60  0000 C CNN
-F 2 "Pin_Headers:Pin_Header_Straight_1x02" H 10950 3200 60  0001 C CNN
+F 2 "poncho_educiaa:bornera1x2" H 10950 3200 60  0001 C CNN
 F 3 "" H 10950 3200 60  0000 C CNN
 	1    11000 3150
@@
 F 0 "J3" H 5950 4250 60  0000 C CNN
 F 1 "TB_1X2" H 6000 3650 60  0000 C CNN
-F 2 "Pin_Headers:Pin_Header_Straight_1x02" H 5900 4000 60  0001 C CNN
+F 2 "poncho_educiaa:bornera1x2" H 5900 4000 60  0001 C CNN
 F 3 "" H 5900 4000 60  0000 C CNN
 	1    5950 3950
@@
 F 0 "J4" H 6876 5060 60  0000 C CNN
 F 1 "TB_1X3" H 6926 4310 60  0000 C CNN
-F 2 "Pin_Headers:Pin_Header_Straight_1x03" H 6826 4810 60  0001 C CNN
+F 2 "poncho_educiaa:bornera1x3" H 6826 4810 60  0001 C CNN
 F 3 "" H 6826 4810 60  0000 C CNN
 	1    6876 4760
@@
 F 0 "J6" H 5500 1200 60  0000 C CNN
 F 1 "TB_1X3" H 5550 450 60  0000 C CNN
-F 2 "Pin_Headers:Pin_Header_Straight_1x03" H 5450 950 60  0001 C CNN
+F 2 "poncho_educiaa:bornera1x3" H 5450 950 60  0001 C CNN
 F 3 "" H 5450 950 60  0000 C CNN
 	1    5500 900
@@
 F 0 "J7" H 5500 2300 60  0000 C CNN
 F 1 "TB_1X3" H 5550 1550 60  0000 C CNN
-F 2 "Pin_Headers:Pin_Header_Straight_1x03" H 5450 2050 60  0001 C CNN
+F 2 "poncho_educiaa:bornera1x3" H 5450 2050 60  0001 C CNN
 F 3 "" H 5450 2050 60  0000 C CNN
 	1    5500 2000
@@
 F 0 "J5" H 8972 5060 60  0000 C CNN
 F 1 "TB_1X3" H 9022 4310 60  0000 C CNN
-F 2 "Pin_Headers:Pin_Header_Straight_1x03" H 8922 4810 60  0001 C CNN
+F 2 "poncho_educiaa:bornera1x3" H 8922 4810 60  0001 C CNN
 F 3 "" H 8922 4810 60  0000 C CNN
 	1    8972 4760
@@
 F 0 "J8" H 8312 6320 60  0000 C CNN
 F 1 "TB_1X2" H 8362 5720 60  0000 C CNN
-F 2 "Pin_Headers:Pin_Header_Straight_1x02" H 8262 6070 60  0001 C CNN
+F 2 "poncho_educiaa:bornera1x2" H 8262 6070 60  0001 C CNN
 F 3 "" H 8262 6070 60  0000 C CNN
 	1    8312 6020
@@
 F 0 "J9" H 6174 7014 60  0000 C CNN
 F 1 "TB_1X2" H 6224 6414 60  0000 C CNN
-F 2 "Pin_Headers:Pin_Header_Straight_1x02" H 6124 6764 60  0001 C CNN
+F 2 "poncho_educiaa:bornera1x2" H 6124 6764 60  0001 C CNN
 F 3 "" H 6124 6764 60  0000 C CNN
 	1    6174 6714
@@
 $EndComp
 $Comp
-L LM7805reg 78051
+L LM7805reg 780511
 U 1 1 5683AD9B
 P 6462 6270
-F 0 "78051" H 6746 6684 60  0000 C CNN
+F 0 "780511" H 6746 6684 60  0000 C CNN
 F 1 "LM7805reg" H 6762 6830 60  0000 C CNN
 F 2 "poncho_educiaa:LM7805" H 6462 6270 60  0001 C CNN

Commit message: Circuito de encendido modificado. Se invirtió el orden regulador/interruptor.
Connections:
- wire segments 332 -> 335
Other:
- moved on the sheet: J9

Commit message: Versión final del PCB.
Parts:
- removed 780511: LM7805reg, poncho_educiaa:LM7805, symbol LM7805reg
- added 7805111: LM7805reg, poncho_educiaa:LM7805, symbol LM7805reg
- added C3: C, Capacitors_ThroughHole:C_Disc_D3_P2.5, symbol C
- added C4: CP, Capacitors_SMD:c_elec_6.3x4.5, symbol CP
Connections:
- wire segments 335 -> 339
Other:
- moved on the sheet: D3, D4, R5, R6
Changed lines of the file:
@@
 L +3.3V #PWR013
 U 1 1 56131FC1
-P 7150 1100
-F 0 "#PWR013" H 7150 950 50  0001 C CNN
-F 1 "+3.3V" H 7150 1240 50  0000 C CNN
-F 2 "" H 7150 1100 60  0000 C CNN
-F 3 "" H 7150 1100 60  0000 C CNN
-	1    7150 1100
+P 6954 1024
+F 0 "#PWR013" H 6954 874 50  0001 C CNN
+F 1 "+3.3V" H 6954 1164 50  0000 C CNN
+F 2 "" H 6954 1024 60  0000 C CNN
+F 3 "" H 6954 1024 60  0000 C CNN
+	1    6954 1024
 	1    0    0    -1
 $EndComp
@@
 L R R5
 U 1 1 5682A717
-P 7400 1450
-F 0 "R5" V 7480 1450 50  0000 C CNN
-F 1 "R" V 7400 1450 50  0000 C CNN
-F 2 "Resistors_ThroughHole:Resistor_Horizontal_RM10mm" V 7330 1450 50  0001 C CNN
-F 3 "" H 7400 1450 50  0000 C CNN
-	1    7400 1450
+P 8032 1466
+F 0 "R5" V 8112 1466 50  0000 C CNN
+F 1 "R" V 8032 1466 50  0000 C CNN
+F 2 "Resistors_ThroughHole:Resistor_Horizontal_RM10mm" V 7962 1466 50  0001 C CNN
+F 3 "" H 8032 1466 50  0000 C CNN
+	1    8032 1466
 	0    1    1    0
 $EndComp
@@
 L R R6
 U 1 1 5682A782
-P 8400 1450
-F 0 "R6" V 8480 1450 50  0000 C CNN
-F 1 "R" V 8400 1450 50  0000 C CNN
-F 2 "Resistors_ThroughHole:Resistor_Horizontal_RM10mm" V 8330 1450 50  0001 C CNN
-F 3 "" H 8400 1450 50  0000 C CNN
-	1    8400 1450
+P 9032 1466
+F 0 "R6" V 9112 1466 50  0000 C CNN
+F 1 "R" V 9032 1466 50  0000 C CNN
+F 2 "Resistors_ThroughHole:Resistor_Horizontal_RM10mm" V 8962 1466 50  0001 C CNN
+F 3 "" H 9032 1466 50  0000 C CNN
+	1    9032 1466
 	0    1    1    0
 $EndComp
@@
 L GND #PWR024
 U 1 1 5682AB63
-P 7000 1900
-F 0 "#PWR024" H 7000 1650 50  0001 C CNN
-F 1 "GND" H 7000 1750 50  0000 C CNN
-F 2 "" H 7000 1900 50  0000 C CNN
-F 3 "" H 7000 1900 50  0000 C CNN
-	1    7000 1900
+P 7632 1916
+F 0 "#PWR024" H 7632 1666 50  0001 C CNN
+F 1 "GND" H 7632 1766 50  0000 C CNN
+F 2 "" H 7632 1916 50  0000 C CNN
+F 3 "" H 7632 1916 50  0000 C CNN
+	1    7632 1916
 	1    0    0    -1
 $EndComp
@@
 L GND #PWR025
 U 1 1 5682ABA9
-P 8000 1900
-F 0 "#PWR025" H 8000 1650 50  0001 C CNN
-F 1 "GND" H 8000 1750 50  0000 C CNN
-F 2 "" H 8000 1900 50  0000 C CNN
-F 3 "" H 8000 1900 50  0000 C CNN
-	1    8000 1900
+P 8632 1916
+F 0 "#PWR025" H 8632 1666 50  0001 C CNN
+F 1 "GND" H 8632 1766 50  0000 C CNN
+F 2 "" H 8632 1916 50  0000 C CNN
+F 3 "" H 8632 1916 50  0000 C CNN
+	1    8632 1916
 	1    0    0    -1
 $EndComp
@@
 L +3.3V #PWR026
 U 1 1 5682B45D
-P 7200 1450
-F 0 "#PWR026" H 7200 1300 50  0001 C CNN
-F 1 "+3.3V" H 7200 1590 50  0000 C CNN
-F 2 "" H 7200 1450 50  0000 C CNN
-F 3 "" H 7200 1450 50  0000 C CNN
-	1    7200 1450
-	1    0    0    -1
-$EndComp
-Text Label 7800 1450 0    60   ~ 0
+P 7832 1466
+F 0 "#PWR026" H 7832 1316 50  0001 C CNN
+F 1 "+3.3V" H 7832 1606 50  0000 C CNN
+F 2 "" H 7832 1466 50  0000 C CNN
+F 3 "" H 7832 1466 50  0000 C CNN
+	1    7832 1466
+	1    0    0    -1
+$EndComp
+Text Label 8432 1466 0    60   ~ 0
 GPIO2
 $Comp
 L LED D3
 U 1 1 5682B8F2
-P 7300 1750
-F 0 "D3" H 7300 1850 50  0000 C CNN
-F 1 "LED" H 7300 1650 50  0000 C CNN
-F 2 "LEDs:LED-3MM" H 7300 1750 50  0001 C CNN
-F 3 "" H 7300 1750 50  0000 C CNN
-	1    7300 1750
+P 7932 1766
+F 0 "D3" H 7932 1866 50  0000 C CNN
+F 1 "LED" H 7932 1666 50  0000 C CNN
+F 2 "LEDs:LED-3MM" H 7932 1766 50  0001 C CNN
+F 3 "" H 7932 1766 50  0000 C CNN
+	1    7932 1766
 	1    0    0    -1
 $EndComp
@@
 L LED D4
 U 1 1 5682B961
-P 8300 1750
-F 0 "D4" H 8300 1850 50  0000 C CNN
-F 1 "LED" H 8300 1650 50  0000 C CNN
-F 2 "LEDs:LED-3MM" H 8300 1750 50  0001 C CNN
-F 3 "" H 8300 1750 50  0000 C CNN
-	1    8300 1750
+P 8932 1766
+F 0 "D4" H 8932 1866 50  0000 C CNN
+F 1 "LED" H 8932 1666 50  0000 C CNN
+F 2 "LEDs:LED-3MM" H 8932 1766 50  0001 C CNN
+F 3 "" H 8932 1766 50  0000 C CNN
+	1    8932 1766
 	1    0    0    -1
 $EndComp
@@
 	1    0    0    -1
 $EndComp
-$Comp
-L LM7805reg 780511
-U 1 1 5683AD9B
-P 7394 6176
-F 0 "780511" H 7678 6590 60  0000 C CNN
-F 1 "LM7805reg" H 7694 6736 60  0000 C CNN
-F 2 "poncho_educiaa:LM7805" H 7394 6176 60  0001 C CNN
-F 3 "" H 7394 6176 60  0000 C CNN
-	1    7394 6176
-	1    0    0    -1
-$EndComp
 Wire Wire Line
 	6300 3850 7900 3850
@@
 Wire Wire Line
 	7350 1000 7900 1000
-Wire Wire Line
-	7150 1100 7900 1100
 Connection ~ 9750 2050
 Wire Wire Line
@@
 	6450 2300 6450 2450
 Wire Wire Line
-	8100 1750 8000 1750
-Wire Wire Line
-	8000 1750 8000 1900
-Wire Wire Line
-	7100 1750 7000 1750
-Wire Wire Line
-	7000 1750 7000 1900
-Wire Wire Line
-	7550 1450 7550 1750
-Wire Wire Line
-	7550 1750 7500 1750
-Wire Wire Line
-	8550 1450 8550 1750
-Wire Wire Line
-	8550 1750 8500 1750
-Wire Wire Line
-	7200 1450 7250 1450
-Wire Wire Line
-	7800 1450 8250 1450
+	8732 1766 8632 1766
+Wire Wire Line
+	8632 1766 8632 1916
+Wire Wire Line
+	7732 1766 7632 1766
+Wire Wire Line
+	7632 1766 7632 1916
+Wire Wire Line
+	8182 1466 8182 1766
+Wire Wire Line
+	8182 1766 8132 1766
+Wire Wire Line
+	9182 1466 9182 1766
+Wire Wire Line
+	9182 1766 9132 1766
+Wire Wire Line
+	7832 1466 7882 1466
+Wire Wire Line
+	8432 1466 8882 1466
 Wire Notes Line
 	8474 5460 11174 5460
@@
 	7872 5920 7962 5920
 Wire Wire Line
-	7962 6120 7962 6386
-Wire Wire Line
-	7962 6386 7604 6386
-Wire Wire Line
 	7456 6388 7292 6388
 Wire Wire Line
@@
 Wire Wire Line
 	7234 6370 7234 6432
+$Comp
+L C C3
+U 1 1 5696F87E
+P 6954 1254
+F 0 "C3" H 6979 1354 50  0000 L CNN
+F 1 "C" H 6979 1154 50  0000 L CNN
+F 2 "Capacitors_ThroughHole:C_Disc_D3_P2.5" H 6992 1104 50  0001 C CNN
+F 3 "" H 6954 1254 50  0000 C CNN
+	1    6954 1254
+	1    0    0    -1
+$EndComp
+$Comp
+L CP C4
+U 1 1 5696F92B
+P 7180 1252
+F 0 "C4" H 7205 1352 50  0000 L CNN
+F 1 "CP" H 7205 1152 50  0000 L CNN
+F 2 "Capacitors_SMD:c_elec_6.3x4.5" H 7218 1102 50  0001 C CNN
+F 3 "" H 7180 1252 50  0000 C CNN
+	1    7180 1252
+	1    0    0    -1
+$EndComp
+Wire Wire Line
+	6954 1100 7900 1100
+Wire Wire Line
+	7180 1100 7180 1102
+Wire Wire Line
+	6954 1024 6954 1104
+Connection ~ 7180 1100
+Connection ~ 6954 1100
+$Comp
+L GND #PWR033
+U 1 1 56970492
+P 6954 1438
+F 0 "#PWR033" H 6954 1188 50  0001 C CNN
+F 1 "GND" H 6954 1288 50  0000 C CNN
+F 2 "" H 6954 1438 50  0000 C CNN
+F 3 "" H 6954 1438 50  0000 C CNN
+	1    6954 1438
+	1    0    0    -1
+$EndComp
+$Comp
+L GND #PWR034
+U 1 1 569704E4
+P 7180 1438
+F 0 "#PWR034" H 7180 1188 50  0001 C CNN
+F 1 "GND" H 7180 1288 50  0000 C CNN
+F 2 "" H 7180 1438 50  0000 C CNN
+F 3 "" H 7180 1438 50  0000 C CNN
+	1    7180 1438
+	1    0    0    -1
+$EndComp
+Wire Wire Line
+	7180 1402 7180 1438
+Wire Wire Line
+	6954 1404 6954 1438
+$Comp
+L LM7805reg 7805111
+U 1 1 56970E58
+P 7394 6176
+F 0 "7805111" H 7678 6590 60  0000 C CNN
+F 1 "LM7805reg" H 7694 6736 60  0000 C CNN
+F 2 "poncho_educiaa:LM7805" H 7394 6176 60  0001 C CNN
+F 3 "" H 7394 6176 60  0000 C CNN
+	1    7394 6176
+	1    0    0    -1
+$EndComp
+Wire Wire Line
+	7604 6386 7962 6386
+Wire Wire Line
+	7962 6386 7962 6120
 Wire Wire Line
 	7234 6432 7604 6432
