File: schematics_&_pcb/poncho.sch (KiCad schematic (older format))
At the start: 31 parts, among them J1 TB_1X2, J2 TB_1X2, J3 TB_1X2, J4 TB_1X3, J5 TB_1X3, J6 TB_1X3, J7 TB_1X3, J8 TB_1X2, J9 TB_1X2, P1 CONN_20X2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

Commit message: Corrección de warnings y rótulos. La aplicación Android se movió al repositorio de SW.
Connections:
- wire segments 339 -> 347
- no-connect marks 6 -> 37
Other:
- note added: "Alimentación"
- note added: "Recepción"
- moved on the sheet: J9
