File: schematics_&_pcb/poncho.kicad_pcb (KiCad board)
At the start: 2 copper layers, 49 parts, among them J1 TB_1X2, J2 TB_1X2, J3 TB_1X2, J4 TB_1X3, J5 TB_1X3, J6 TB_1X3, J7 TB_1X3, J8 TB_1X2, J9 TB_1X2, P1 CONN_20X2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

Commit message: Circuito de encendido modificado. Se invirtió el orden regulador/interruptor.
Parts:
- moved 780511 9.00 mm to (143.6, 38.0), turned to 0 degrees
- moved J8 7.53 mm to (153.4, 42.0), turned to 270 degrees
- moved SW1 4.85 mm to (137.1, 47.4)
Connections:
- J8 pad 1: Net-(J8-Pad1) -> Net-(780511-Pad3)
- J9 pad 1: Net-(780511-Pad1) -> Net-(J9-Pad1)
- SW1 pad 1: Net-(J8-Pad1) -> Net-(780511-Pad1)
- SW1 pad 2: Net-(780511-Pad3) -> Net-(J9-Pad1)
Routing:
- net Net-(J9-Pad1): track 0.00 -> 5.88 mm
- net Net-(J8-Pad1): track 3.75 -> 0.00 mm
- net Net-(780511-Pad2): track 28.8 -> 30.9 mm
- net Net-(780511-Pad3): track 5.69 -> 6.67 mm
- net Net-(780511-Pad1): track 4.81 -> 5.40 mm
Changed lines of the file:
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@@
     (links 112)
     (no_connects 14)
-    (area 46.249999 31.585 252.169491 122.889919)
+    (area 0 0 0 0)
     (thickness 1.6)
     (drawings 18)
-    (tracks 315)
+    (tracks 321)
     (zones 0)
     (modules 49)
@@
   (net 62 "Net-(R4-Pad2)")
   (net 63 "Net-(R7-Pad1)")
-  (net 64 "Net-(J8-Pad1)")
-  (net 65 "Net-(SW1-Pad4)")
-  (net 66 "Net-(SW1-Pad5)")
-  (net 67 "Net-(SW1-Pad6)")
-  (net 68 "Net-(SW1-Pad3)")
-  (net 69 "Net-(780511-Pad1)")
-  (net 70 "Net-(780511-Pad2)")
-  (net 71 "Net-(780511-Pad3)")
+  (net 64 "Net-(SW1-Pad4)")
+  (net 65 "Net-(SW1-Pad5)")
+  (net 66 "Net-(SW1-Pad6)")
+  (net 67 "Net-(SW1-Pad3)")
+  (net 68 "Net-(780511-Pad1)")
+  (net 69 "Net-(780511-Pad2)")
+  (net 70 "Net-(780511-Pad3)")
+  (net 71 "Net-(J9-Pad1)")
   (net_class Default "This is the default net class."
     (clearance 0.25)
@@
     (add_net "Net-(D3-Pad2)")
     (add_net "Net-(D4-Pad2)")
-    (add_net "Net-(J8-Pad1)")
+    (add_net "Net-(J9-Pad1)")
     (add_net "Net-(R1-Pad2)")
     (add_net "Net-(R2-Pad1)")
@@
   )
   (module poncho_educiaa:6pin_switch (layer F.Cu)
-    (at 141.88 46.74)
+    (at 137.08 47.4)
     (fp_text reference SW1 (at 13.86 -5.23) (layer F.SilkS)
       (effects (font (size 1 1) (thickness 0.15)))
@@
     (fp_line (start 3.5 -6) (end 3.5 1.5) (layer F.SilkS) (width 0.15))
     (pad 4 thru_hole circle (at 10 0) (size 2.2 2.2) (drill 0.75) (layers *.Cu *.Mask F.SilkS)
-      (net 65 "Net-(SW1-Pad4)"))
+      (net 64 "Net-(SW1-Pad4)"))
     (pad 5 thru_hole circle (at 10 -2.4) (size 2.2 2.2) (drill 0.75) (layers *.Cu *.Mask F.SilkS)
-      (net 66 "Net-(SW1-Pad5)"))
+      (net 65 "Net-(SW1-Pad5)"))
     (pad 6 thru_hole circle (at 10 -4.8) (size 2.2 2.2) (drill 0.75) (layers *.Cu *.Mask F.SilkS)
-      (net 67 "Net-(SW1-Pad6)"))
+      (net 66 "Net-(SW1-Pad6)"))
     (pad 3 thru_hole circle (at 5 0) (size 2.2 2.2) (drill 0.75) (layers *.Cu *.Mask F.SilkS)
-      (net 68 "Net-(SW1-Pad3)"))
+      (net 67 "Net-(SW1-Pad3)"))
     (pad 2 thru_hole circle (at 5 -2.4) (size 2.2 2.2) (drill 0.75) (layers *.Cu *.Mask F.SilkS)
-      (net 71 "Net-(780511-Pad3)"))
+      (net 71 "Net-(J9-Pad1)"))
     (pad 1 thru_hole circle (at 5 -4.8) (size 2.2 2.2) (drill 0.75) (layers *.Cu *.Mask F.SilkS)
-      (net 64 "Net-(J8-Pad1)"))
+      (net 68 "Net-(780511-Pad1)"))
   )
   (module poncho_educiaa:LM7805 (layer F.Cu)
-    (at 141.71 46.85 90)
-    (fp_text reference 780511 (at -1.87 -12.68 90) (layer F.SilkS)
-      (effects (font (size 1 1) (thickness 0.15)))
-    )
-    (fp_text value LM7805reg (at -2 -14.71 90) (layer F.Fab)
+    (at 143.58 38.05)
+    (fp_text reference 780511 (at -1.87 -12.68) (layer F.SilkS)
+      (effects (font (size 1 1) (thickness 0.15)))
+    )
+    (fp_text value LM7805reg (at -2 -14.71) (layer F.Fab)
       (effects (font (size 1 1) (thickness 0.15)))
     )
@@
     (fp_line (start 7.2 1) (end -2.4 1) (layer F.SilkS) (width 0.15))
     (fp_line (start -2.4 1.65) (end 7.2 1.65) (layer F.SilkS) (width 0.15))
-    (pad 1 thru_hole circle (at 0 0 90) (size 2.2 2.2) (drill 0.75) (layers *.Cu *.Mask F.SilkS)
-      (net 69 "Net-(780511-Pad1)"))
-    (pad 2 thru_hole circle (at 2.4 0 90) (size 2.2 2.2) (drill 0.75) (layers *.Cu *.Mask F.SilkS)
-      (net 70 "Net-(780511-Pad2)"))
-    (pad 3 thru_hole circle (at 4.8 0 90) (size 2.2 2.2) (drill 0.75) (layers *.Cu *.Mask F.SilkS)
-      (net 71 "Net-(780511-Pad3)"))
+    (pad 1 thru_hole circle (at 0 0) (size 2.2 2.2) (drill 0.75) (layers *.Cu *.Mask F.SilkS)
+      (net 68 "Net-(780511-Pad1)"))
+    (pad 2 thru_hole circle (at 2.4 0) (size 2.2 2.2) (drill 0.75) (layers *.Cu *.Mask F.SilkS)
+      (net 69 "Net-(780511-Pad2)"))
+    (pad 3 thru_hole circle (at 4.8 0) (size 2.2 2.2) (drill 0.75) (layers *.Cu *.Mask F.SilkS)
+      (net 70 "Net-(780511-Pad3)"))
   )
   (module poncho_educiaa:bornera1x2 (layer F.Cu)
-    (at 146.87 38.26)
-    (fp_text reference J8 (at 4 -4.5) (layer F.SilkS)
-      (effects (font (size 1 1) (thickness 0.15)))
-    )
-    (fp_text value TB_1X2 (at 4 -5.5) (layer F.Fab)
+    (at 153.42 41.98 270)
+    (fp_text reference J8 (at 4 -4.5 270) (layer F.SilkS)
+      (effects (font (size 1 1) (thickness 0.15)))
+    )
+    (fp_text value TB_1X2 (at 4 -5.5 270) (layer F.Fab)
       (effects (font (size 1 1) (thickness 0.15)))
     )
@@
     (fp_line (start 6.5 -2) (end -2 -2) (layer F.SilkS) (width 0.15))
     (fp_line (start -2 -2) (end -2 2) (layer F.SilkS) (width 0.15))
-    (pad 1 thru_hole rect (at 0 0) (size 3 3) (drill 1) (layers *.Cu *.Mask F.SilkS)
-      (net 64 "Net-(J8-Pad1)"))
-    (pad 2 thru_hole circle (at 5 0) (size 3 3) (drill 1) (layers *.Cu *.Mask F.SilkS)
-      (net 70 "Net-(780511-Pad2)"))
+    (pad 1 thru_hole rect (at 0 0 270) (size 3 3) (drill 1) (layers *.Cu *.Mask F.SilkS)
+      (net 70 "Net-(780511-Pad3)"))
+    (pad 2 thru_hole circle (at 5 0 270) (size 3 3) (drill 1) (layers *.Cu *.Mask F.SilkS)
+      (net 69 "Net-(780511-Pad2)"))
   )
   (module poncho_educiaa:bornera1x2 (layer F.Cu)
@@
     (fp_line (start -2 -2) (end -2 2) (layer F.SilkS) (width 0.15))
     (pad 1 thru_hole rect (at 0 0 90) (size 3 3) (drill 1) (layers *.Cu *.Mask F.SilkS)
-      (net 69 "Net-(780511-Pad1)"))
+      (net 71 "Net-(J9-Pad1)"))
     (pad 2 thru_hole circle (at 5 0 90) (size 3 3) (drill 1) (layers *.Cu *.Mask F.SilkS)
-      (net 70 "Net-(780511-Pad2)"))
+      (net 69 "Net-(780511-Pad2)"))
   )
   (module poncho_educiaa:bornera1x3 (layer F.Cu)
@@
   (segment (start 231.55 71.6) (end 235.96 71.6) (width 1) (layer B.Cu) (net 63))
   (segment (start 235.96 71.6) (end 235.97 71.59) (width 1) (layer B.Cu) (net 63))
-  (segment (start 146.88 38.2) (end 146.88 41.94) (width 1) (layer B.Cu) (net 64))
-  (segment (start 146.89 38.21) (end 146.88 38.2) (width 1) (layer B.Cu) (net 64))
-  (segment (start 141.59 46.93) (end 141.68 46.84) (width 1) (layer B.Cu) (net 69))
-  (segment (start 136.91 46.93) (end 141.59 46.93) (width 1) (layer B.Cu) (net 69))
-  (segment (start 137.02 41.99) (end 137.02 36.6) (width 1) (layer B.Cu) (net 70))
-  (segment (start 151.87 36.28) (end 151.87 38.26) (width 1) (layer B.Cu) (net 70))
-  (segment (start 151.18 35.59) (end 151.87 36.28) (width 1) (layer B.Cu) (net 70))
-  (segment (start 138.03 35.59) (end 151.18 35.59) (width 1) (layer B.Cu) (net 70))
-  (segment (start 137.02 36.6) (end 138.03 35.59) (width 1) (layer B.Cu) (net 70))
-  (segment (start 141.71 44.45) (end 139.48 44.45) (width 1) (layer B.Cu) (net 70))
-  (segment (start 139.48 44.45) (end 137.02 41.99) (width 1) (layer B.Cu) (net 70))
-  (segment (start 151.87 38.26) (end 151.87 38.12) (width 1) (layer B.Cu) (net 70))
-  (segment (start 141.68 42.04) (end 144.19 43.06) (width 1) (layer B.Cu) (net 71))
-  (segment (start 144.19 43.06) (end 146.88 44.34) (width 1) (layer B.Cu) (net 71))
+  (segment (start 142.08 42.6) (end 142.08 39.55) (width 1) (layer B.Cu) (net 68) (status 400000))
+  (segment (start 142.08 39.55) (end 143.58 38.05) (width 1) (layer B.Cu) (net 68) (status 800000))
+  (segment (start 143.42 38.21) (end 143.58 38.05) (width 1) (layer B.Cu) (net 68))
+  (segment (start 153.42 46.98) (end 151.81 46.98) (width 1) (layer B.Cu) (net 69) (status 400000))
+  (segment (start 145.98 39.75) (end 145.98 38.05) (width 1) (layer B.Cu) (net 69) (status 800000))
+  (segment (start 146.54 40.31) (end 145.98 39.75) (width 1) (layer B.Cu) (net 69))
+  (segment (start 148.67 40.31) (end 146.54 40.31) (width 1) (layer B.Cu) (net 69))
+  (segment (start 149.72 41.36) (end 148.67 40.31) (width 1) (layer B.Cu) (net 69))
+  (segment (start 149.72 44.89) (end 149.72 41.36) (width 1) (layer B.Cu) (net 69))
+  (segment (start 151.81 46.98) (end 149.72 44.89) (width 1) (layer B.Cu) (net 69))
+  (segment (start 137.02 41.99) (end 137.02 37.66) (width 1) (layer B.Cu) (net 69))
+  (segment (start 145.98 36.03) (end 145.98 38.05) (width 1) (layer B.Cu) (net 69))
+  (segment (start 145.08 35.13) (end 145.98 36.03) (width 1) (layer B.Cu) (net 69))
+  (segment (start 139.55 35.13) (end 145.08 35.13) (width 1) (layer B.Cu) (net 69))
+  (segment (start 137.02 37.66) (end 139.55 35.13) (width 1) (layer B.Cu) (net 69))
+  (segment (start 148.38 38.05) (end 149.49 38.05) (width 1) (layer B.Cu) (net 70) (status 400000))
+  (segment (start 149.49 38.05) (end 153.42 41.98) (width 1) (layer B.Cu) (net 70) (status 800000))
+  (segment (start 137.02 46.99) (end 137.97 46.99) (width 1) (layer B.Cu) (net 71) (status C00000))
+  (segment (start 137.97 46.99) (end 139.96 45) (width 1) (layer B.Cu) (net 71) (status 400000))
+  (segment (start 139.96 45) (end 142.08 45) (width 1) (layer B.Cu) (net 71) (status 800000))
   (zone (net 4) (net_name GND) (layer F.Cu) (hatch edge 0.508)
     (connect_pads (clearance 0.508))

Commit message: Versión final del PCB.
Parts:
- added C3: C, Capacitors_ThroughHole:C_Disc_D3_P2.5, F.Cu at (138.4, 61.2)
- added C4: C, Capacitors_ThroughHole:C_Disc_D3_P2.5, F.Cu at (131.8, 61.2)
- added REF**: SolderWirePad_single_2mmDrill, Wire_Pads:SolderWirePad_single_2mmDrill, F.Cu at (137.1, 67.5)
Connections:
- J8 pad 1: Net-(780511-Pad3) -> Net-(7805111-Pad3)
- J8 pad 2: Net-(780511-Pad2) -> Net-(7805111-Pad2)
- J9 pad 2: Net-(780511-Pad2) -> Net-(7805111-Pad2)
- SW1 pad 1: Net-(780511-Pad1) -> Net-(7805111-Pad1)
Routing:
- net GND: track 109.8 -> 123.8 mm
- net Net-(780511-Pad2): track 30.9 -> 25.0 mm
- net Net-(7805111-Pad2): track 0.00 -> 5.94 mm
- net Net-(7805111-Pad3): track 0.00 -> 5.56 mm
- net Net-(780511-Pad3): track 6.67 -> 1.11 mm
- net Net-(7805111-Pad1): track 0.00 -> 3.05 mm
- net Net-(780511-Pad1): track 5.40 -> 2.35 mm
- net (no net): track 944.5 -> 942.0 mm
Other:
- board text added: "D"
- board text added: "E"

Commit message: Corrección de warnings y rótulos. La aplicación Android se movió al repositorio de SW.
Other:
- board text added: "PCB del regulador de 5V, en caso que sea necesario el uso del mismo."
Changed lines of the file:
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@@
-(kicad_pcb (version 4) (host pcbnew 4.0.1-3.201512221402+6198~38~ubuntu14.04.1-stable)
+(kicad_pcb (version 4) (host pcbnew 4.0.2-4+6225~38~ubuntu14.04.1-stable)
   (general
     (links 113)
@@
     (area 45.599999 32.469999 252.169491 122.889919)
     (thickness 1.6)
-    (drawings 35)
+    (drawings 41)
     (tracks 323)
     (zones 0)
@@
   )
   (page A4)
+  (title_block
+    (title "Poncho de control de motores por Wi-Fi")
+    (date 2016-02-16)
+    (rev 1.1)
+    (company "UNLP - Cátedra de Taller de Proyecto 1 - Grupo 1: Ailán, Bouche, Hourquebie, Liotta")
+    (comment 1 "Poncho para Computadora Industrial Abierta Argentina Versión Educativa EDU-CIAA-NXP")
+    (comment 2 "Licencia: https://github.com/ciaa/Hardware/tree/master/Readme (LICENSE)")
+  )
   (layers
     (0 F.Cu power)
@@
     )
   )
+  (gr_line (start 121.34 24.41) (end 121.37 24.41) (angle 90) (layer B.Adhes) (width 0.2))
+  (gr_line (start 121.34 31.73) (end 121.34 24.41) (angle 90) (layer B.Adhes) (width 0.2))
+  (gr_line (start 169.79 31.73) (end 121.34 31.73) (angle 90) (layer B.Adhes) (width 0.2))
+  (gr_line (start 169.79 24.37) (end 169.79 31.73) (angle 90) (layer B.Adhes) (width 0.2))
+  (gr_line (start 121.45 24.37) (end 169.79 24.37) (angle 90) (layer B.Adhes) (width 0.2))
+  (gr_text "PCB del regulador de 5V, en caso que \nsea necesario el uso del mismo." (at 146.47 28.11) (layer B.Adhes)
+    (effects (font (size 1.5 1.5) (thickness 0.3)))
+  )
   (gr_text + (at 154.84 38.6) (layer B.Cu)
